File: KaControl3.sch (KiCad schematic (older format))
At the start: 30 parts

Commit message: Various changes
Parts:
- gave numbers to parts that had none: 30
Connections:
- net SW: now reaches U1.4 (SENSOR_VP)
- net EMAC_RXD0 renamed ETH_RXD0
- net EMAC_RXD1 renamed ETH_RXD1
- net EMAC_RX_DV renamed ETH_CRS_DV
- net EMAC_TXD0 renamed ETH_TXD0
- net EMAC_TXD1 renamed ETH_TXD1
- net EMAC_TX_CLK renamed ETH_REF_CLK
- net EMAC_TX_EN renamed ETH_TX_EN
- net I2C_SCL renamed SCL1
- net I2C_SDA renamed SDA1
- net PHY_POWER renamed ETH_POWER
Other:
- note added: "DBG-Ausgabe in Firmware deaktivieren\nund Pins für GSM nutzen?"
- note added: "SW(4) für \n"Analog Keyboard"?"
- note added: "Zur Einsparung von Pins: I2C statt SPI \nfür KaBus (Verbindung zum IO-Board) nutzen\n--> +2 bzw +4 Pins!"
